Commit message: added gripper and camera

File: igus_rebel/urdf/igus_rebel.description.xacro (robot description, xacro)
@@ -1,226 +1,235 @@
 <?xml version="1.0"?>
 <robot xmlns:xacro="http://wiki.ros.org/xacro" name="igus_rebel_description">
-  <xacro:property name="damping" value="0.1"/>
-  <xacro:property name="friction" value="10.0"/>
-<!-- measured from model -->
-  <link name="base_link">
-    <visual>
-      <geometry>
-        <mesh filename="file://$(find igus_rebel)/meshes/robolink_rebel/Robolink_RebeL_000.dae"/>
-      </geometry>
-    </visual>
-    <collision>
-      <geometry>
-        <mesh filename="file://$(find igus_rebel)/meshes/robolink_rebel/Robolink_RebeL_000.dae"/>
-      </geometry>
-    </collision>
-    <inertial>
-      <mass value="1.0" />
-      <inertia ixx="1.0" iyy="1.0" izz="1.0" ixy="0.0" ixz="0.0" iyz="0.0" />
-    </inertial>
-  </link>
-  <joint name="joint1" type="revolute">
-    <parent link="base_link"/>
-    <child link="link_1"/>
-    <origin rpy="0.0 0.0 ${pi}" xyz="0.0 0 0.126"/>
-    <axis xyz="0 0 -1"/>
-    <limit effort="330.0" lower="${-pi*179/180}" upper="${pi*179/180}" velocity="${pi*45/180}"/> <!-- limit taken from the controller -->
-    <dynamics damping="${damping}" friction="${friction}"/>
-  </joint>
-  <link name="link_1">
-    <visual>
-      <geometry>
-        <mesh filename="file://$(find igus_rebel)/meshes/robolink_rebel/Robolink_RebeL_001.dae"/>
-      </geometry>
-      <origin rpy="0 0 ${pi}" xyz="0.0 0.0 -0.0537"/>
-    </visual>
-    <collision>
-      <geometry>
-        <mesh filename="file://$(find igus_rebel)/meshes/robolink_rebel/Robolink_RebeL_001.dae"/>
-      </geometry>
-      <origin rpy="0 0 ${pi}" xyz="0.0 0.0 -0.0537"/>
-    </collision>
-    <inertial>
-      <mass value="0.1" />
-      <inertia ixx="0.03" iyy="0.03" izz="0.03" ixy="0.0" ixz="0.0" iyz="0.0" />
-    </inertial>
-  </link>
-  <joint name="joint2" type="revolute">
-    <parent link="link_1"/>
-    <child link="link_2"/>
-    <origin rpy="0.0 0.0 0.0" xyz="0.0 0.025 0.153"/>
-    <axis xyz="0 -1 0"/>
-    <limit effort="330.0" lower="${-pi*11/18}" upper="${pi*11/18}" velocity="${pi*45/180}"/> <!-- limits taken from the controller -->
-    <dynamics damping="${damping}" friction="${friction}"/>
-  </joint>
-  <link name="link_2">
-    <visual>
-      <geometry>
-        <mesh filename="file://$(find igus_rebel)/meshes/robolink_rebel/Robolink_RebeL_002_0.dae"/>
-      </geometry>
-      <origin rpy="-1.5707 0 0" xyz="0 -0.005 -0.00625"/>
-    </visual>
-    <collision>
-      <geometry>
-        <mesh filename="file://$(find igus_rebel)/meshes/robolink_rebel/Robolink_RebeL_002_0.dae"/>
-      </geometry>
-      <origin rpy="-1.5707 0 0" xyz="0 -0.005 -0.00625"/>
-    </collision>
-    <inertial>
-      <mass value="0.1" />
-      <inertia ixx="0.03" iyy="0.03" izz="0.03" ixy="0.0" ixz="0.0" iyz="0.0" />
-    </inertial>
-  </link>
-  <joint name="joint_fixed_1" type="fixed">
-    <parent link="link_2"/>
-    <child link="link_3"/>
-    <origin rpy="0.0 0.0 0.0" xyz="0.0 -0.025 0.1"/>
-    <dynamics damping="${damping}" friction="${friction}"/>
-  </joint>
-  <link name="link_3">
-    <visual>
-      <geometry>
-        <mesh filename="file://$(find igus_rebel)/meshes/robolink_rebel/Robolink_RebeL_002_1.dae"/>
-      </geometry>
-      <origin rpy="0 0 ${pi}" xyz="0 -0.00625 -0.00625"/>
-    </visual>
-    <collision>
-      <geometry>
-        <mesh filename="file://$(find igus_rebel)/meshes/robolink_rebel/Robolink_RebeL_002_1.dae"/>
-      </geometry>
-      <origin rpy="0 0 ${pi}" xyz="0 -0.00625 -0.00625"/>
-    </collision>
-    <inertial>
-      <mass value="0.1" />
-      <inertia ixx="0.03" iyy="0.03" izz="0.03" ixy="0.0" ixz="0.0" iyz="0.0" />
-    </inertial>
-  </link>
-  <joint name="joint_fixed_2" type="fixed">
-    <parent link="link_3"/>
-    <child link="link_4"/>
-		<origin rpy="0.0 -1.0 0.0" xyz="-0.035 0.003 0.055" />
-    <dynamics damping="${damping}" friction="${friction}"/>
-  </joint>
-    <link name="link_4">
-    <visual>
-      <geometry>
-        <mesh filename="file://$(find igus_rebel)/meshes/robolink_rebel/Robolink_RebeL_002_2.dae"/>
-      </geometry>
-      <origin rpy="0 0 ${-pi}" xyz="0.0 0.0 -0.00625"/>
-    </visual>
-    <collision>
-      <geometry>
-        <mesh filename="file://$(find igus_rebel)/meshes/robolink_rebel/Robolink_RebeL_002_2.dae"/>
-      </geometry>
-      <origin rpy="0 0 ${-pi}" xyz="0.0 0.0 -0.00625"/>
-    </collision>
-    <inertial>
-      <mass value="0.1" />
-      <inertia ixx="0.03" iyy="0.03" izz="0.03" ixy="0.0" ixz="0.0" iyz="0.0" />
-    </inertial>
-  </link>
-    <joint name="joint3" type="revolute">
-    <parent link="link_4"/>
-    <child link="link_5"/>
-		<origin rpy="0.0 0 0.0" xyz="0.005 0.015 0.096" />
-    <axis xyz="0 -1 0"/>
-    <limit effort="330.0" lower="${-pi*11/18}" upper="${pi*11/18}" velocity="${pi*45/180}"/>
-    <dynamics damping="${damping}" friction="${friction}"/>
-  </joint>
-  <link name="link_5">
-    <visual>
-      <geometry>
-        <mesh filename="file://$(find igus_rebel)/meshes/robolink_rebel/Robolink_RebeL_003.dae"/>
-      </geometry>
-      <origin rpy="-1.5707 0 0" xyz="0 -0.008 -0.008"/>
-    </visual>
-    <collision>
-      <geometry>
-        <mesh filename="file://$(find igus_rebel)/meshes/robolink_rebel/Robolink_RebeL_003.dae"/>
-      </geometry>
-      <origin rpy="-1.5707 0 0" xyz="0 -0.008 -0.008"/>
-    </collision>
-    <inertial>
-      <mass value="0.1" />
-      <inertia ixx="0.03" iyy="0.03" izz="0.03" ixy="0.0" ixz="0.0" iyz="0.0" />
-    </inertial>
-  </link>
-  <joint name="joint4" type="revolute">
-    <parent link="link_5"/>
-    <child link="link_6"/>
-		<origin rpy="-0.05 0.0 0.0" xyz="0.0 -0.025 0.145" />
-    <axis xyz="0 0 1"/>
-    <limit effort="330.0" lower="${-pi*179/180}" upper="${pi*179/180}" velocity="${pi*45/180}"/>
-    <dynamics damping="${damping}" friction="${friction}"/>
-  </joint>
-  <link name="link_6">
-    <visual>
-      <geometry>
-        <mesh filename="file://$(find igus_rebel)/meshes/robolink_rebel/Robolink_RebeL_004.dae"/>
-      </geometry>
-      <origin rpy="0 0 0" xyz="0 0 -0.003125"/>
-    </visual>
-    <collision>
-      <geometry>
-        <mesh filename="file://$(find igus_rebel)/meshes/robolink_rebel/Robolink_RebeL_004.dae"/>
-      </geometry>
-      <origin rpy="0 0 0" xyz="0 0 -0.003125"/>
-    </collision>
-    <inertial>
-      <mass value="0.1" />
-      <inertia ixx="0.03" iyy="0.03" izz="0.03" ixy="0.0" ixz="0.0" iyz="0.0" />
-    </inertial>
-  </link>
-  <joint name="joint5" type="revolute">
-    <parent link="link_6"/>
-    <child link="link_7"/>
-    <origin rpy="0.0 0.0 0.0" xyz="0.0 0.029 0.143"/>
-    <axis xyz="0 -1 0"/>
-		<limit effort="330.0" lower="${-pi*19/36}" upper="${pi*19/36}" velocity="${pi*45/180}" />
-    <dynamics damping="${damping}" friction="${friction}"/>
-  </joint>
-  <link name="link_7">
-    <visual>
-      <geometry>
-        <mesh filename="file://$(find igus_rebel)/meshes/robolink_rebel/Robolink_RebeL_005.dae"/>
-      </geometry>
-      <origin rpy="0 1.57 -1.5707" xyz="0 -0.00625 0"/>
-    </visual>
-    <collision>
-      <geometry>
-        <mesh filename="file://$(find igus_rebel)/meshes/robolink_rebel/Robolink_RebeL_005.dae"/>
-      </geometry>
-      <origin rpy="0 1.57 -1.5707" xyz="0 -0.00625 0"/>
-    </collision>
-    <inertial>
-      <mass value="0.1" />
-      <inertia ixx="0.03" iyy="0.03" izz="0.03" ixy="0.0" ixz="0.0" iyz="0.0" />
-    </inertial>
-  </link>
-  <joint name="joint6" type="revolute">
-    <parent link="link_7"/>
-    <child link="link_8"/>
-    <origin rpy="0.0 0.0 0.0" xyz="0.0 -0.029 0.1188"/>
-    <axis xyz="0 0 1"/>
-		<limit effort="330.0" lower="${-pi*179/180}" upper="${pi*179/180}" velocity="${pi*45/180}" />
-    <dynamics damping="${damping}" friction="${friction}"/>
-  </joint>
-  <link name="link_8">
-    <visual>
-      <geometry>
-        <mesh filename="file://$(find igus_rebel)/meshes/robolink_rebel/Robolink_RebeL_006.dae"/>
-      </geometry>
-      <origin rpy="0 -1.57 0" xyz="0.0 0.0 -0.00625"/>
-    </visual>
-    <collision>
-      <geometry>
-        <mesh filename="file://$(find igus_rebel)/meshes/robolink_rebel/Robolink_RebeL_006.dae"/>
-      </geometry>
-      <origin rpy="0 -1.57 0" xyz="0.0 0.0 -0.00625"/>
-    </collision>
-    <inertial>
-      <mass value="0.1" />
-      <inertia ixx="0.03" iyy="0.03" izz="0.03" ixy="0.0" ixz="0.0" iyz="0.0" />
-    </inertial>
-  </link>
+  <xacro:macro name="igus_rebel_description">
+    <xacro:property name="damping" value="0.1"/>
+    <xacro:property name="friction" value="10.0"/>
+    <link name="base_link">
+      <visual>
+        <geometry>
+          <mesh filename="file://$(find igus_rebel)/meshes/robolink_rebel/Robolink_RebeL_000.dae"/>
+        </geometry>
+      </visual>
+      <collision>
+        <geometry>
+          <mesh filename="file://$(find igus_rebel)/meshes/robolink_rebel/Robolink_RebeL_000.dae"/>
+        </geometry>
+      </collision>
+      <inertial>
+        <mass value="1.0" />
+        <inertia ixx="1.0" iyy="1.0" izz="1.0" ixy="0.0" ixz="0.0" iyz="0.0" />
+      </inertial>
+    </link>
+    <joint name="joint1" type="revolute">
+      <parent link="base_link"/>
+      <child link="link_1"/>
+      <origin rpy="0.0 0.0 ${pi}" xyz="0.0 0 0.126"/>
+      <axis xyz="0 0 -1"/>
+      <limit effort="330.0" lower="${-pi*179/180}" upper="${pi*179/180}" velocity="${pi*45/180}"/> <!-- limit taken from the controller -->
+      <dynamics damping="${damping}" friction="${friction}"/>
+    </joint>
+    <link name="link_1">
+      <visual>
+        <geometry>
+          <mesh filename="file://$(find igus_rebel)/meshes/robolink_rebel/Robolink_RebeL_001.dae"/>
+        </geometry>
+        <origin rpy="0 0 ${pi}" xyz="0.0 0.0 -0.0537"/>
+      </visual>
+      <collision>
+        <geometry>
+          <mesh filename="file://$(find igus_rebel)/meshes/robolink_rebel/Robolink_RebeL_001.dae"/>
+        </geometry>
+        <origin rpy="0 0 ${pi}" xyz="0.0 0.0 -0.0537"/>
+      </collision>
+      <inertial>
+        <mass value="0.1" />
+        <inertia ixx="0.03" iyy="0.03" izz="0.03" ixy="0.0" ixz="0.0" iyz="0.0" />
+      </inertial>
+    </link>
+    <joint name="joint2" type="revolute">
+      <parent link="link_1"/>
+      <child link="link_2"/>
+      <origin rpy="0.0 0.0 0.0" xyz="0.0 0.025 0.153"/>
+      <axis xyz="0 -1 0"/>
+      <limit effort="330.0" lower="${-pi*11/18}" upper="${pi*11/18}" velocity="${pi*45/180}"/> <!-- limits taken from the controller -->
+      <dynamics damping="${damping}" friction="${friction}"/>
+    </joint>
+    <link name="link_2">
+      <visual>
+        <geometry>
+          <mesh filename="file://$(find igus_rebel)/meshes/robolink_rebel/Robolink_RebeL_002_0.dae"/>
+        </geometry>
+        <origin rpy="-1.5707 0 0" xyz="0 -0.005 -0.00625"/>
+      </visual>
+      <collision>
+        <geometry>
+          <mesh filename="file://$(find igus_rebel)/meshes/robolink_rebel/Robolink_RebeL_002_0.dae"/>
+        </geometry>
+        <origin rpy="-1.5707 0 0" xyz="0 -0.005 -0.00625"/>
+      </collision>
+      <inertial>
+        <mass value="0.1" />
+        <inertia ixx="0.03" iyy="0.03" izz="0.03" ixy="0.0" ixz="0.0" iyz="0.0" />
+      </inertial>
+    </link>
+    <joint name="joint_fixed_1" type="fixed">
+      <parent link="link_2"/>
+      <child link="link_3"/>
+      <origin rpy="0.0 0.0 0.0" xyz="0.0 -0.025 0.1"/>
+      <dynamics damping="${damping}" friction="${friction}"/>
+    </joint>
+    <link name="link_3">
+      <visual>
+        <geometry>
+          <mesh filename="file://$(find igus_rebel)/meshes/robolink_rebel/Robolink_RebeL_002_1.dae"/>
+        </geometry>
+        <origin rpy="0 0 ${pi}" xyz="0 -0.00625 -0.00625"/>
+      </visual>
+      <collision>
+        <geometry>
+          <mesh filename="file://$(find igus_rebel)/meshes/robolink_rebel/Robolink_RebeL_002_1.dae"/>
+        </geometry>
+        <origin rpy="0 0 ${pi}" xyz="0 -0.00625 -0.00625"/>
+      </collision>
+      <inertial>
+        <mass value="0.1" />
+        <inertia ixx="0.03" iyy="0.03" izz="0.03" ixy="0.0" ixz="0.0" iyz="0.0" />
+      </inertial>
+    </link>
+    <joint name="joint_fixed_2" type="fixed">
+      <parent link="link_3"/>
+      <child link="link_4"/>
+      <origin rpy="0.0 -1.0 0.0" xyz="-0.035 0.003 0.055" />
+      <dynamics damping="${damping}" friction="${friction}"/>
+    </joint>
+      <link name="link_4">
+      <visual>
+        <geometry>
+          <mesh filename="file://$(find igus_rebel)/meshes/robolink_rebel/Robolink_RebeL_002_2.dae"/>
+        </geometry>
+        <origin rpy="0 0 ${-pi}" xyz="0.0 0.0 -0.00625"/>
+      </visual>
+      <collision>
+        <geometry>
+          <mesh filename="file://$(find igus_rebel)/meshes/robolink_rebel/Robolink_RebeL_002_2.dae"/>
+        </geometry>
+        <origin rpy="0 0 ${-pi}" xyz="0.0 0.0 -0.00625"/>
+      </collision>
+      <inertial>
+        <mass value="0.1" />
+        <inertia ixx="0.03" iyy="0.03" izz="0.03" ixy="0.0" ixz="0.0" iyz="0.0" />
+      </inertial>
+    </link>
+      <joint name="joint3" type="revolute">
+      <parent link="link_4"/>
+      <child link="link_5"/>
+      <origin rpy="0.0 0 0.0" xyz="0.005 0.015 0.096" />
+      <axis xyz="0 -1 0"/>
+      <limit effort="330.0" lower="${-pi*11/18}" upper="${pi*11/18}" velocity="${pi*45/180}"/>
+      <dynamics damping="${damping}" friction="${friction}"/>
+    </joint>
+    <link name="link_5">
+      <visual>
+        <geometry>
+          <mesh filename="file://$(find igus_rebel)/meshes/robolink_rebel/Robolink_RebeL_003.dae"/>
+        </geometry>
+        <origin rpy="-1.5707 0 0" xyz="0 -0.008 -0.008"/>
+      </visual>
+      <collision>
+        <geometry>
+          <mesh filename="file://$(find igus_rebel)/meshes/robolink_rebel/Robolink_RebeL_003.dae"/>
+        </geometry>
+        <origin rpy="-1.5707 0 0" xyz="0 -0.008 -0.008"/>
+      </collision>
+      <inertial>
+        <mass value="0.1" />
+        <inertia ixx="0.03" iyy="0.03" izz="0.03" ixy="0.0" ixz="0.0" iyz="0.0" />
+      </inertial>
+    </link>
+    <joint name="joint4" type="revolute">
+      <parent link="link_5"/>
+      <child link="link_6"/>
+      <origin rpy="-0.05 0.0 0.0" xyz="0.0 -0.025 0.145" />
+      <axis xyz="0 0 1"/>
+      <limit effort="330.0" lower="${-pi*179/180}" upper="${pi*179/180}" velocity="${pi*45/180}"/>
+      <dynamics damping="${damping}" friction="${friction}"/>
+    </joint>
+    <link name="link_6">
+      <visual>
+        <geometry>
+          <mesh filename="file://$(find igus_rebel)/meshes/robolink_rebel/Robolink_RebeL_004.dae"/>
+        </geometry>
+        <origin rpy="0 0 0" xyz="0 0 -0.003125"/>
+      </visual>
+      <collision>
+        <geometry>
+          <mesh filename="file://$(find igus_rebel)/meshes/robolink_rebel/Robolink_RebeL_004.dae"/>
+        </geometry>
+        <origin rpy="0 0 0" xyz="0 0 -0.003125"/>
+      </collision>
+      <inertial>
+        <mass value="0.1" />
+        <inertia ixx="0.03" iyy="0.03" izz="0.03" ixy="0.0" ixz="0.0" iyz="0.0" />
+      </inertial>
+    </link>
+    <joint name="joint5" type="revolute">
+      <parent link="link_6"/>
+      <child link="link_7"/>
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
File: igus_rebel/urdf/igus_rebel.gazebo.xacro (robot description, xacro)
@@ -2,4 +2,7 @@
 <robot xmlns:xacro="http://www.ros.org/wiki/xacro" name="igus_rebel_gazebo">
     <!-- Gazebo requires the use of plugins to interact with other systems such as ROS. -->
+    <gazebo reference="camera_mount">
+        <material>Gazebo/Green</material>
+    </gazebo>
     <!-- This plugin will publish the joint_states for the selected joints
             (which robot_state_publisher can then use to broadcast the approprate tf). -->

File: igus_rebel/urdf/igus_rebel.urdf.xacro (robot description, xacro)
@@ -1,9 +1,12 @@
 <?xml version="1.0"?>
 <robot xmlns:xacro="http://wiki.ros.org/xacro" name="igus_rebel" >
-  <!-- igus_rebel -->
+  <xacro:arg name="gripper" default="none" />
   <xacro:include filename="$(find igus_rebel)/urdf/igus_rebel.description.xacro"/>
+  <xacro:igus_rebel_description  />
   <xacro:include filename="$(find igus_rebel)/urdf/igus_rebel.control.xacro"/>
   <xacro:include filename="$(find igus_rebel)/urdf/igus_rebel.gazebo.xacro"/>
   <xacro:igus_rebel_control arm_id="igus_rebel"/>
+  <xacro:include filename="$(find igus_rebel)/urdf/grippers.xacro"/>
+  <xacro:gripper gripper_type="$(arg gripper)" />
   <link name="world" />
   <joint name="world_joint" type="fixed">

File: igus_rebel/urdf/igus_rebel_ros2.urdf.xacro (robot description, xacro)
@@ -1,4 +1,5 @@
 <?xml version="1.0"?>
 <robot xmlns:xacro="http://wiki.ros.org/xacro" name="igus_rebel_ros2" >
+  <xacro:arg name="gripper" default="none" />
   <xacro:include filename="$(find igus_rebel)/urdf/igus_rebel_ros2.description.xacro"/>
   <xacro:igus_rebel_ros2_description  />
@@ -6,4 +7,6 @@
   <xacro:include filename="$(find igus_rebel)/urdf/igus_rebel.gazebo.xacro"/>
   <xacro:igus_rebel_control arm_id="igus_rebel_ros2"/>
+  <xacro:include filename="$(find igus_rebel)/urdf/grippers.xacro"/>
+  <xacro:gripper gripper_type="$(arg gripper)" />
   <link name="world" />
   <joint name="world_joint" type="fixed">
