Commit message: removed Realsense camera

File: igus_rebel/urdf/grippers.xacro (robot description, xacro)
@@ -45,13 +45,4 @@
             </joint>
             <link name="camera_insert" />
-            <!-- includes the realsense D435 ros2 description file and its collision box-->
-            <xacro:arg name="use_nominal_extrinsics" default="false" />
-            <xacro:arg name="add_plug" default="true" />
-            <xacro:arg name="use_mesh" default="true" />
-            <xacro:include filename="$(find igus_rebel)/urdf/camera/_d435.urdf.xacro" />
-            <xacro:sensor_d435 parent="camera_insert" use_nominal_extrinsics="$(arg use_nominal_extrinsics)"
-                add_plug="$(arg add_plug)" use_mesh="$(arg use_mesh)">
-                <origin xyz="0.0 0 0" rpy="0 0 0" />
-            </xacro:sensor_d435>
         </xacro:if>
     </xacro:macro>

Commit message: added OAK D Pro camera, and show data on Rviz

File: igus_rebel/urdf/grippers.xacro (robot description, xacro)
@@ -45,4 +45,9 @@
             </joint>
             <link name="camera_insert" />
+            <joint name="camera_insert_to_oakd" type="fixed">
+                <parent link="camera_insert"/>
+                <child link="oakd"/>
+                <origin xyz="0.03 0.005 0.0155" rpy="0 0 0"/>
+            </joint>
         </xacro:if>
     </xacro:macro>

File: igus_rebel/urdf/igus_rebel.urdf.xacro (robot description, xacro)
@@ -5,8 +5,10 @@
   <xacro:igus_rebel_description  />
   <xacro:include filename="$(find igus_rebel)/urdf/igus_rebel.control.xacro"/>
-  <xacro:include filename="$(find igus_rebel)/urdf/igus_rebel.gazebo.xacro"/>
   <xacro:igus_rebel_control arm_id="igus_rebel"/>
   <xacro:include filename="$(find igus_rebel)/urdf/grippers.xacro"/>
-  <xacro:gripper gripper_type="$(arg gripper)" />
+  <xacro:gripper gripper_type="$(arg gripper)"/>
+  <xacro:include filename="$(find igus_rebel)/urdf/camera/oak_d_pro.xacro"/>
+  <xacro:oakd_link/>
+  <xacro:include filename="$(find igus_rebel)/urdf/igus_rebel.gazebo.xacro"/>
   <link name="world" />
   <joint name="world_joint" type="fixed">

File: igus_rebel/urdf/igus_rebel_ros2.urdf.xacro (robot description, xacro)
@@ -3,10 +3,12 @@
   <xacro:arg name="gripper" default="none" />
   <xacro:include filename="$(find igus_rebel)/urdf/igus_rebel_ros2.description.xacro"/>
-  <xacro:igus_rebel_ros2_description  />
+  <xacro:igus_rebel_ros2_description/>
   <xacro:include filename="$(find igus_rebel)/urdf/igus_rebel.control.xacro"/>
-  <xacro:include filename="$(find igus_rebel)/urdf/igus_rebel.gazebo.xacro"/>
   <xacro:igus_rebel_control arm_id="igus_rebel_ros2"/>
   <xacro:include filename="$(find igus_rebel)/urdf/grippers.xacro"/>
-  <xacro:gripper gripper_type="$(arg gripper)" />
+  <xacro:gripper gripper_type="$(arg gripper)"/>
+  <xacro:include filename="$(find igus_rebel)/urdf/camera/oak_d_pro.xacro"/>
+  <xacro:oakd_link/>
+  <xacro:include filename="$(find igus_rebel)/urdf/igus_rebel.gazebo.xacro"/>
   <link name="world" />
   <joint name="world_joint" type="fixed">
