Commit message: added gazebo ignition package

File: igus_rebel_description_ros2/urdf/camera/oak_d_pro.xacro (robot description, xacro)
@@ -2,5 +2,5 @@
 <!--  xacro macros for oakd mount -->
 <robot name="oak_d_pro" xmlns:xacro="http://ros.org/wiki/xacro">
-    <xacro:include filename="$(find igus_rebel_description)/urdf/common_properties.urdf.xacro"/>
+    <xacro:include filename="$(find igus_rebel_description_ros2)/urdf/common_properties.urdf.xacro"/>
     <xacro:macro name="inertial_box" params="mass x y z *origin">
         <inertial>
@@ -25,5 +25,5 @@
             <visual>
                 <geometry>
-                    <mesh filename="file://$(find igus_rebel_description)/meshes/camera/OAK-D_pro.dae"/>
+                    <mesh filename="file://$(find igus_rebel_description_ros2)/meshes/camera/OAK-D_pro.dae"/>
                 </geometry>
             </visual>
@@ -189,64 +189,4 @@
             <preserveFixedJoint>true</preserveFixedJoint>
         </gazebo>
-        <!-- FOR GZ CLASSIC -->
-        <!-- <gazebo reference="oakd">
-            <sensor type="depth" name="oakd_depth">
-                <always_on>1</always_on>
-                <update_rate>15</update_rate>
-                <camera name="oakd_d_camera">
-                    <horizontal_fov>2.21</horizontal_fov>
-                    <image>
-                        <width>1280</width>
-                        <height>800</height>
-                        <format>B8G8R8</format>
-                    </image>
-                    <clip>
-                        <near>0.05</near>
-                        <far>8.0</far>
-                    </clip>
-                </camera>
-                <plugin name="depth_driver_plugin" filename="libgazebo_ros_camera.so">
-                    <ros>
-                        <namespace></namespace>
-                    </ros>
-                    <camera_name>oakd_depth</camera_name>
-                    <frame_name>camera_optical_frame</frame_name>
-                    <hack_baseline>0.07</hack_baseline>
-                    <min_depth>0.01</min_depth>
-                    <max_depth>9.0</max_depth>
-                </plugin>
-            </sensor>
-        </gazebo>
-        <gazebo reference="oakd">
-            <material>Gazebo/Black</material>
-            <sensor type="camera" name="oakd_rgb">
-                <visualize>true</visualize>
-                <update_rate>30.0</update_rate>
-                <camera name="oakd_rgb_camera">
-                    <horizontal_fov>2.21</horizontal_fov>
-                    <image>
-                        <width>1280</width>
-                        <height>800</height>
-                        <format>R8G8B8</format>
-                    </image>
-                    <clip>
-                        <near>0.03</near>
-                        <far>300</far>
-                    </clip>
-                    <noise>
-                        <type>gaussian</type>
-                        <mean>0.0</mean>
-                        <stddev>0.007</stddev>
-                    </noise>
-                </camera>
-                <plugin name="camera_controller" filename="libgazebo_ros_camera.so">
-                    <camera_name>oakd_rgb</camera_name>
-                    <frame_name>camera_optical_frame</frame_name>
-                    <ros>
-                        <namespace>oakd_rgb</namespace>
-                    </ros>
-                </plugin>
-            </sensor>
-        </gazebo> -->
     </xacro:macro>
 </robot>

File: igus_rebel_description_ros2/urdf/igus_rebel.gazebo.xacro (robot description, xacro)
@@ -59,31 +59,7 @@
                 <i_min>1.0</i_min>
         </plugin>
-        <!-- <plugin filename="ignition-gazebo-sensors-system" name="ignition::gazebo::systems::Sensors">
+        <plugin filename="ignition-gazebo-sensors-system" name="ignition::gazebo::systems::Sensors">
             <render_engine>ogre2</render_engine>
-        </plugin> -->
-    </gazebo>
-    <!-- <gazebo>
-        <plugin name="gazebo_ros_joint_state_publisher"
-            filename="libgazebo_ros_joint_state_publisher.so">
-            <update_rate>20</update_rate>
-            <joint_name>joint1</joint_name>
-            <joint_name>joint2</joint_name>
-            <joint_name>joint3</joint_name>
-            <joint_name>joint4</joint_name>
-            <joint_name>joint5</joint_name>
-            <joint_name>joint6</joint_name>
         </plugin>
     </gazebo>
-    <gazebo>
-        <plugin name="gazebo_ros_joint_pose_trajectory"
-            filename="libgazebo_ros_joint_pose_trajectory.so">
-            <update_rate>2</update_rate>
-        </plugin>
-    </gazebo> -->
 </robot>
-    <!-- This plugin will read a JointTrajectory message from the /set_joint_trajectory topic
-            and move the machine accordingly. It's a bit clunky but it works. -->
-    <!-- You'll probably want to add damping to the joints to stop them it flopping around.
-            e.g. <dynamics damping="10.0" friction="10.0"/> -->
-    <!-- Here's an example message to publish to test it:
-            ros2 topic pub -1 /set_joint_trajectory trajectory_msgs/msg/JointTrajectory  '{header: {frame_id: world}, joint_names: [slider_joint, arm_joint], points: [  {positions: {0.8,0.6}} ]}' -->

Commit message: added use sim time control on visualize and moveit launch, oakd_link is now camera_link, added clock bridge,  corrected ignition launch

File: igus_rebel_description_ros2/urdf/camera/oak_d_pro.xacro (robot description, xacro)
@@ -19,8 +19,8 @@
         <joint name="camera_insert_to_oakd" type="fixed">
             <parent link="camera_insert"/>
-            <child link="oakd_link"/>
+            <child link="camera_link"/>
             <origin xyz="0.03 0.005 0.0155" rpy="0 0 0"/>
         </joint>
-        <link name="oakd_link">
+        <link name="camera_link">
             <visual>
                 <geometry>
@@ -42,5 +42,5 @@
         </link>
         <joint name="oakd_depth_camera_joint" type="fixed">
-            <parent link="oakd_link"/>
+            <parent link="camera_link"/>
             <child link="oakd_depth_camera_frame"/>
             <origin xyz="0 0 0" rpy="0 0 0" />
@@ -58,5 +58,5 @@
         </link>
         <joint name="oakd_rgb_camera_joint" type="fixed">
-            <parent link="oakd_link"/>
+            <parent link="camera_link"/>
             <child link="oakd_rgb_camera_frame"/>
             <origin xyz="0 0 0" rpy="0 0 0" />
@@ -74,5 +74,5 @@
         </link>
         <joint name="oakd_left_camera_joint" type="fixed">
-            <parent link="oakd_link"/>
+            <parent link="camera_link"/>
             <child link="oakd_left_camera_frame"/>
             <origin xyz="0 0.0375 0" rpy="0 0 0" />
@@ -90,5 +90,5 @@
         </link>
         <joint name="oakd_right_camera_joint" type="fixed">
-            <parent link="oakd_link"/>
+            <parent link="camera_link"/>
             <child link="oakd_right_camera_frame"/>
             <origin xyz="0 -0.0375 0" rpy="0 0 0" />
@@ -106,5 +106,5 @@
         </link>
         <joint name="oakd_imu_joint" type="fixed">
-            <parent link="oakd_link"/>
+            <parent link="camera_link"/>
             <child link="oakd_imu_frame"/>
             <origin xyz="0 0 0" rpy="-1.5707963267948966 0 -1.5707963267948966" />
@@ -154,6 +154,6 @@
                     <horizontal_fov>1.05</horizontal_fov>
                     <image>
-                        <width>1280</width>
-                        <height>720</height>
+                        <width>320</width>
+                        <height>240</height>
                         <format>R8G8B8</format>
                     </image>
