Commit message: adjusted some argument checks, and folders

File: igus_rebel_description_ros2/urdf/camera/oak_d_pro_camera.xacro (robot description, xacro)
@@ -25,5 +25,5 @@
             <visual>
                 <geometry>
-                    <mesh filename="file://$(find igus_rebel_description_ros2)/meshes/camera/oak_d_pro_camera.dae"/>
+                    <mesh filename="file://$(find igus_rebel_description_ros2)/meshes/cameras/oak_d_pro_camera.dae"/>
                 </geometry>
             </visual>

File: igus_rebel_description_ros2/urdf/grippers/grippers.xacro (robot description, xacro)
@@ -23,5 +23,5 @@
                 <origin xyz="0.008 0 0" rpy="0 0 ${pi}" />
                 <geometry>
-                    <mesh filename="file://$(find igus_rebel_description_ros2)/meshes/camera_mount.stl"
+                    <mesh filename="file://$(find igus_rebel_description_ros2)/meshes/mounts/camera_mount.stl"
                         scale="0.001 0.001 0.001" />
                 </geometry>
@@ -31,5 +31,5 @@
                 <origin xyz="0.008 0 0" rpy="0 0 ${pi}" />
                 <geometry>
-                    <mesh filename="file://$(find igus_rebel_description_ros2)/meshes/camera_mount.stl"
+                    <mesh filename="file://$(find igus_rebel_description_ros2)/meshes/mounts/camera_mount.stl"
                         scale="0.001 0.001 0.001" />
                 </geometry>

File: igus_rebel_description_ros2/urdf/igus_rebel/igus_rebel.description.xacro (robot description, xacro)
@@ -2,5 +2,5 @@
 <robot xmlns:xacro="http://www.ros.org/wiki/xacro" name="igus_rebel">
     <material name="dark_grey">
-        <color rgba="${2/255} ${2/255} ${2/255} 1.0" />
+        <color rgba="${5/255} ${5/255} ${5/255} 1.0" />
     </material>
     <xacro:macro name="igus_rebel_description">
@@ -11,11 +11,11 @@
             <visual>
                 <geometry>
-                    <mesh filename="file://$(find igus_rebel_description_ros2)/meshes/new/Joint0.dae" />
-                </geometry>
-                <material name="dark_grey"/>
-            </visual>
-            <collision>
-                <geometry>
-                    <mesh filename="file://$(find igus_rebel_description_ros2)/meshes/new/Joint0.dae" />
+                    <mesh filename="file://$(find igus_rebel_description_ros2)/meshes/igus_rebel/Joint0.dae" />
+                </geometry>
+                <material name="dark_grey"/>
+            </visual>
+            <collision>
+                <geometry>
+                    <mesh filename="file://$(find igus_rebel_description_ros2)/meshes/igus_rebel/Joint0.dae" />
                 </geometry>
             </collision>
@@ -36,12 +36,12 @@
             <visual>
                 <geometry>
-                    <mesh filename="file://$(find igus_rebel_description_ros2)/meshes/new/Joint1.dae" />
-                </geometry>
-                <origin rpy="0 0 0" xyz="0 0 0" />
-                <material name="dark_grey"/>
-            </visual>
-            <collision>
-                <geometry>
-                    <mesh filename="file://$(find igus_rebel_description_ros2)/meshes/new/Joint1.dae" />
+                    <mesh filename="file://$(find igus_rebel_description_ros2)/meshes/igus_rebel/Joint1.dae" />
+                </geometry>
+                <origin rpy="0 0 0" xyz="0 0 0" />
+                <material name="dark_grey"/>
+            </visual>
+            <collision>
+                <geometry>
+                    <mesh filename="file://$(find igus_rebel_description_ros2)/meshes/igus_rebel/Joint1.dae" />
                 </geometry>
                 <origin rpy="0 0 0" xyz="0 0 0" />
@@ -64,12 +64,12 @@
             <visual>
                 <geometry>
-                    <mesh filename="file://$(find igus_rebel_description_ros2)/meshes/new/Joint2.dae" />
-                </geometry>
-                <origin rpy="0 0 0" xyz="0 0 0" />
-                <material name="dark_grey"/>
-            </visual>
-            <collision>
-                <geometry>
-                    <mesh filename="file://$(find igus_rebel_description_ros2)/meshes/new/Joint2.dae" />
+                    <mesh filename="file://$(find igus_rebel_description_ros2)/meshes/igus_rebel/Joint2.dae" />
+                </geometry>
+                <origin rpy="0 0 0" xyz="0 0 0" />
+                <material name="dark_grey"/>
+            </visual>
+            <collision>
+                <geometry>
+                    <mesh filename="file://$(find igus_rebel_description_ros2)/meshes/igus_rebel/Joint2.dae" />
                 </geometry>
                 <origin rpy="0 0 0" xyz="0 0 0" />
@@ -92,12 +92,12 @@
             <visual>
                 <geometry>
-                    <mesh filename="file://$(find igus_rebel_description_ros2)/meshes/new/Joint3.dae" />
-                </geometry>
-                <origin rpy="0 0 0" xyz="0 0 0" />
-                <material name="dark_grey"/>
-            </visual>
-            <collision>
-                <geometry>
-                    <mesh filename="file://$(find igus_rebel_description_ros2)/meshes/new/Joint3.dae" />
+                    <mesh filename="file://$(find igus_rebel_description_ros2)/meshes/igus_rebel/Joint3.dae" />
+                </geometry>
+                <origin rpy="0 0 0" xyz="0 0 0" />
+                <material name="dark_grey"/>
+            </visual>
+            <collision>
+                <geometry>
+                    <mesh filename="file://$(find igus_rebel_description_ros2)/meshes/igus_rebel/Joint3.dae" />
                 </geometry>
                 <origin rpy="0 0 0" xyz="0 0 0" />
@@ -120,12 +120,12 @@
             <visual>
                 <geometry>
-                    <mesh filename="file://$(find igus_rebel_description_ros2)/meshes/new/Joint4.dae" />
-                </geometry>
-                <origin rpy="0 0 0" xyz="0 0 0" />
-                <material name="dark_grey"/>
-            </visual>
-            <collision>
-                <geometry>
-                    <mesh filename="file://$(find igus_rebel_description_ros2)/meshes/new/Joint4.dae" />
+                    <mesh filename="file://$(find igus_rebel_description_ros2)/meshes/igus_rebel/Joint4.dae" />
+                </geometry>
+                <origin rpy="0 0 0" xyz="0 0 0" />
+                <material name="dark_grey"/>
+            </visual>
+            <collision>
+                <geometry>
+                    <mesh filename="file://$(find igus_rebel_description_ros2)/meshes/igus_rebel/Joint4.dae" />
                 </geometry>
                 <origin rpy="0 0 0" xyz="0 0 0" />
@@ -148,12 +148,12 @@
             <visual>
                 <geometry>
-                    <mesh filename="file://$(find igus_rebel_description_ros2)/meshes/new/Joint5.dae" />
-                </geometry>
-                <origin rpy="0 0 0" xyz="0 0 0" />
-                <material name="dark_grey"/>
-            </visual>
-            <collision>
-                <geometry>
-                    <mesh filename="file://$(find igus_rebel_description_ros2)/meshes/new/Joint5.dae" />
+                    <mesh filename="file://$(find igus_rebel_description_ros2)/meshes/igus_rebel/Joint5.dae" />
+                </geometry>
+                <origin rpy="0 0 0" xyz="0 0 0" />
+                <material name="dark_grey"/>
+            </visual>
+            <collision>
+                <geometry>
+                    <mesh filename="file://$(find igus_rebel_description_ros2)/meshes/igus_rebel/Joint5.dae" />
                 </geometry>
                 <origin rpy="0 0 0" xyz="0 0 0" />
@@ -175,5 +175,5 @@
             <visual>
                 <geometry>
-                    <mesh filename="file://$(find igus_rebel_description_ros2)/meshes/new/Joint6.dae" />
+                    <mesh filename="file://$(find igus_rebel_description_ros2)/meshes/igus_rebel/Joint6.dae" />
                 </geometry>
                 <origin rpy="0 0 0" xyz="0.0 0 0" />
@@ -182,5 +182,5 @@
             <collision>
                 <geometry>
-                    <mesh filename="file://$(find igus_rebel_description_ros2)/meshes/new/Joint6.dae" />
+                    <mesh filename="file://$(find igus_rebel_description_ros2)/meshes/igus_rebel/Joint6.dae" />
                 </geometry>
                 <origin rpy="0 0 0" xyz="0.0 0 0" />
@@ -198,6 +198,5 @@
             <dynamics damping="${damping}" friction="${friction}"/>
         </joint>
-        <link name="flange">
-        </link>
+        <link name="flange"></link>
     </xacro:macro>
 </robot>

File: igus_rebel_description_ros2/urdf/igus_rebel/igus_rebel.gazebo.xacro (robot description, xacro)
@@ -23,87 +23,66 @@
     </xacro:macro>
     <!-- Sensor plugin -->
-    <gazebo>
-        <plugin filename="ignition-gazebo-sensors-system" name="ignition::gazebo::systems::Sensors">
-            <render_engine>ogre2</render_engine>
-        </plugin>
-    </gazebo>
-    <gazebo reference="virtual_rgb_camera_frame">
-        <sensor type="camera" name="rgb_camera">
-            <camera>
-                <horizontal_fov>1.05</horizontal_fov>
-                <image>
-                    <width>1280</width>
-                    <height>720</height>
-                </image>
-                <clip>
-                    <near>0.3</near>
-                    <far>100</far>
-                </clip>
-                <optical_frame_id>virtual_rgb_camera_frame</optical_frame_id>
-            </camera>
-            <always_on>1</always_on>
-            <update_rate>30</update_rate>
-            <visualize>true</visualize>
-        </sensor>
-    </gazebo>
-    <gazebo reference="virtual_depth_camera_frame">
-        <sensor type="rgbd_camera" name="depth_camera">
-            <update_rate>10</update_rate>
-            <depth_camera>
-                <horizontal_fov>1.05</horizontal_fov>
-                <image>
-                    <width>320</width>
-                    <height>240</height>
-                    <!-- <width>1280</width>
-                    <height>720</height> -->
-                    <format>R8G8B8</format>
-                </image>
-                <clip>
-                    <near>0.1</near>
-                    <far>10.0</far>
-                </clip>
-            </depth_camera>
-        </sensor>
-    </gazebo>
-    <gazebo reference="virtual_depth_camera_frame">
-        <sensor type="rgbd_camera" name="pointcloud">
-            <update_rate>10</update_rate>
-            <camera>
-                <horizontal_fov>1.05</horizontal_fov>
-                <image>
-                    <width>320</width>
-                    <height>240</height>
-                    <format>R8G8B8</format>
-                </image>
-                <clip>
-                    <near>0.1</near>
-                    <far>10.0</far>
-                </clip>
-            </camera>
-        </sensor>
-    </gazebo>
-    <!-- <gazebo reference="oakd_joint">
-        <preserveFixedJoint>true</preserveFixedJoint>
-    </gazebo>
-    <gazebo reference="oakd_rgb_camera_joint">
-        <preserveFixedJoint>true</preserveFixedJoint>
-    </gazebo>
-    <gazebo reference="oakd_rgb_camera_optical_joint">
-        <preserveFixedJoint>true</preserveFixedJoint>
-    </gazebo>
-    <gazebo reference="oakd_left_camera_joint">
-        <preserveFixedJoint>true</preserveFixedJoint>
-    </gazebo>
-    <gazebo reference="oakd_left_camera_optical_joint">
-        <preserveFixedJoint>true</preserveFixedJoint>
-    </gazebo>
-    <gazebo reference="oakd_right_camera_joint">
-        <preserveFixedJoint>true</preserveFixedJoint>
-    </gazebo>
-    <gazebo reference="oakd_right_camera_optical_joint">
-        <preserveFixedJoint>true</preserveFixedJoint>
-    </gazebo>
-    <gazebo reference="oakd_imu_joint">
-        <preserveFixedJoint>true</preserveFixedJoint>
-    </gazebo> -->
+    <xacro:macro name="virtual_sensors">
+        <gazebo>
+            <plugin filename="ignition-gazebo-sensors-system" name="ignition::gazebo::systems::Sensors">
+                <render_engine>ogre2</render_engine>
+            </plugin>
+        </gazebo>
+        <!-- Sensor for RGB, depth and pointcloud data -->
+        <gazebo reference="virtual_rgb_camera_frame">
+            <sensor type="camera" name="rgb_camera">
+                <camera>
+                    <horizontal_fov>1.05</horizontal_fov>
+                    <image>
+                        <width>1280</width>
+                        <height>720</height>
+                    </image>
+                    <clip>
+                        <near>0.3</near>
+                        <far>100</far>
+                    </clip>
+                    <optical_frame_id>virtual_rgb_camera_frame</optical_frame_id>
+                </camera>
+                <always_on>1</always_on>
+                <update_rate>30</update_rate>
+                <visualize>true</visualize>
+            </sensor>
+        </gazebo>
+        <gazebo reference="virtual_depth_camera_frame">
+            <sensor type="rgbd_camera" name="depth_camera">
+                <update_rate>10</update_rate>
+                <depth_camera>
+                    <horizontal_fov>1.05</horizontal_fov>
+                    <image>
+                        <width>320</width>
+                        <height>240</height>
+                        <!-- <width>1280</width>
+                        <height>720</height> -->
+                        <format>R8G8B8</format>
+                    </image>
+                    <clip>
+                        <near>0.1</near>
+                        <far>10.0</far>
+                    </clip>
+                </depth_camera>
+            </sensor>
+        </gazebo>
+        <gazebo reference="virtual_depth_camera_frame">
+            <sensor type="rgbd_camera" name="pointcloud">
+                <update_rate>10</update_rate>
+                <camera>
+                    <horizontal_fov>1.05</horizontal_fov>
+                    <image>
+                        <width>320</width>
+                        <height>240</height>
+                        <format>R8G8B8</format>
+                    </image>
+                    <clip>
+                        <near>0.1</near>
+                        <far>10.0</far>
+                    </clip>
+                </camera>
+            </sensor>
+        </gazebo>
+    </xacro:macro>
 </robot>

File: igus_rebel_description_ros2/urdf/igus_rebel/igus_rebel.urdf.xacro (robot description, xacro)
@@ -23,4 +23,7 @@
                 <xacro:ign_joint_state_publisher/>
             </xacro:unless>
+            <xacro:unless value="${camera == 'none' or gripper == 'none'}">
+                <xacro:virtual_sensors/>
+            </xacro:unless>
         </xacro:if>
     </xacro:macro>

File: igus_rebel_description_ros2/urdf/robot.urdf.xacro (robot description, xacro)
@@ -7,5 +7,5 @@
     <xacro:arg name="gripper" default="none" />
     <!-- Camera type selection -->
-    <xacro:arg name="camera" default="realsense" />
+    <xacro:arg name="camera" default="none" />
     <!-- End effector type selection -->
     <xacro:arg name="end_effector" default="none" />
@@ -15,5 +15,5 @@
     <xacro:arg name="hardware_protocol" default="simulation" />
     <!-- Argument that tells if Moveit2 is used or not -->
-    <xacro:arg name="moveit" default="true" />
+    <xacro:arg name="moveit" default="false" />
     <!-- odometry source: world ground truth or wheels encoders -->
     <xacro:arg name="odometry_source" default="ground_truth" />
