Commit message: hardware interface for Ingition using ign_ros2_contrl plugin works to move the Ingition robot from Moveit2

File: igus_rebel_description_ros2/urdf/igus_rebel/igus_rebel.control.xacro (robot description, xacro)
@@ -19,7 +19,11 @@
 					name="port">3920</param>-->
 				</xacro:if>
+				<xacro:if value="${hardware_protocol == 'ignition'}">
+					<plugin>ign_ros2_control/IgnitionSystem</plugin>
+				</xacro:if>
 			</hardware>
 			<xacro:macro name="rebel_joint" params="name position_min=0 position_max=0 cri_joint_offset=0">
 				<joint name="${name}">
+					<param name="initial_position">0.0</param>
 					<!--<command_interface name="position">
 						<param name="min">${position_min}</param>

File: igus_rebel_description_ros2/urdf/igus_rebel/igus_rebel.gazebo.xacro (robot description, xacro)
@@ -1,7 +1,93 @@
 <?xml version="1.0"?>
 <robot xmlns:xacro="http://www.ros.org/wiki/xacro" name="igus_rebel_gazebo">
+    <xacro:macro name="ign_ros2_control" params="controller_parameters">
+        <gazebo>
+            <plugin filename="ign_ros2_control-system" name="ign_ros2_control::IgnitionROS2ControlPlugin">
+                <parameters>${controller_parameters}</parameters>
+            </plugin>
+        </gazebo>
+    </xacro:macro>
+    <gazebo reference="igus_rebel_base_link">
+        <mu1 value="1.0"/>
+        <mu2 value="1.0"/>
+        <self_collide>false</self_collide>
+    </gazebo>
+    <gazebo reference="link_1">
+        <mu1 value="1.0"/>
+        <mu2 value="1.0"/>
+        <self_collide>false</self_collide>
+    </gazebo>
+    <gazebo reference="link_2">
+        <mu1 value="1.0"/>
+        <mu2 value="1.0"/>
+        <self_collide>false</self_collide>
+    </gazebo>
+    <gazebo reference="link_5">
+        <mu1 value="1.0"/>
+        <mu2 value="1.0"/>
+        <self_collide>false</self_collide>
+    </gazebo>
+    <gazebo reference="link_6">
+        <mu1 value="1.0"/>
+        <mu2 value="1.0"/>
+        <self_collide>false</self_collide>
+    </gazebo>
+    <gazebo reference="link_7">
+        <mu1 value="1.0"/>
+        <mu2 value="1.0"/>
+        <self_collide>false</self_collide>
+    </gazebo>
+    <gazebo reference="link_8">
+        <mu1 value="1.0"/>
+        <mu2 value="1.0"/>
+        <self_collide>false</self_collide>
+    </gazebo>
+    <gazebo reference="joint1">
+        <springStiffness value="0.0"/>
+        <springReference value="0.0"/>
+        <preserveFixedJoint>false</preserveFixedJoint>
+        <disableFixedJointLumping>false</disableFixedJointLumping>
+    </gazebo>
+    <gazebo reference="joint2">
+        <springStiffness value="0.0"/>
+        <springReference value="0.0"/>
+        <preserveFixedJoint>false</preserveFixedJoint>
+        <disableFixedJointLumping>false</disableFixedJointLumping>
+    </gazebo>
+    <gazebo reference="joint3">
+        <springStiffness value="0.0"/>
+        <springReference value="0.0"/>
+        <preserveFixedJoint>false</preserveFixedJoint>
+        <disableFixedJointLumping>false</disableFixedJointLumping>
+    </gazebo>
+    <gazebo reference="joint4">
+        <springStiffness value="0.0"/>
+        <springReference value="0.0"/>
+        <preserveFixedJoint>false</preserveFixedJoint>
+        <disableFixedJointLumping>false</disableFixedJointLumping>
+    </gazebo>
+    <gazebo reference="joint5">
+        <springStiffness value="0.0"/>
+        <springReference value="0.0"/>
+        <preserveFixedJoint>false</preserveFixedJoint>
+        <disableFixedJointLumping>false</disableFixedJointLumping>
+    </gazebo>
+    <gazebo reference="joint6">
+        <springStiffness value="0.0"/>
+        <springReference value="0.0"/>
+        <preserveFixedJoint>false</preserveFixedJoint>
+        <disableFixedJointLumping>false</disableFixedJointLumping>
+    </gazebo>
     <!--joint state publisher-->
     <gazebo>
-        <plugin filename="ignition-gazebo-joint-state-publisher-system" name="ignition::gazebo::systems::JointStatePublisher">
+        <!-- <plugin filename="ignition-gazebo-joint-position-controller-system" name="ignition::gazebo::systems::JointPositionController">
+            <joint_name>joint1</joint_name>
+            <topic>/model/igus_rebel/joint/joint1/0/cmd_pos/data</topic>
+        </plugin> -->
+        <!-- <plugin filename="ignition-gazebo-joint-controller-system" name="ignition::gazebo::systems::JointController">
+                <joint_name>joint1</joint_name>
+                <topic>/model/igus_rebel/joint/joint1/cmd_vel</topic>
+        </plugin> -->
+        <!-- <plugin filename="ignition-gazebo-joint-state-publisher-system" name="ignition::gazebo::systems::JointStatePublisher">
             <joint_name>joint1</joint_name>
             <joint_name>joint2</joint_name>
@@ -10,6 +96,39 @@
             <joint_name>joint5</joint_name>
             <joint_name>joint6</joint_name>
+        </plugin> -->
+        <!-- <plugin filename="ignition-gazebo-joint-trajectory-controller-system" name="ignition::gazebo::systems::JointTrajectoryController">
+            <joint_name>joint1</joint_name>
+            <joint_name>joint2</joint_name>
+            <joint_name>joint3</joint_name>
+            <joint_name>joint4</joint_name>
+            <joint_name>joint5</joint_name>
+            <joint_name>joint6</joint_name>
+            <topic>/model/igus_rebel/joint_trajectory</topic>
+        </plugin> -->
+        <!-- <plugin filename="gz-sim-joint-controller-system" name="gz::sim::systems::JointController">
+            <joint_name>joint1</joint_name>
+            <initial_velocity>5.0</initial_velocity>
         </plugin>
-        <plugin filename="ignition-gazebo-joint-position-controller-system" name="ignition::gazebo::systems::JointPositionController">
+        <plugin filename="gz-sim-joint-controller-system" name="gz::sim::systems::JointController">
+            <joint_name>joint2</joint_name>
+            <initial_velocity>5.0</initial_velocity>
+        </plugin>
+        <plugin filename="gz-sim-joint-controller-system" name="gz::sim::systems::JointController">
+            <joint_name>joint3</joint_name>
+            <initial_velocity>5.0</initial_velocity>
+        </plugin>
+        <plugin filename="gz-sim-joint-controller-system" name="gz::sim::systems::JointController">
+            <joint_name>joint4</joint_name>
+            <initial_velocity>5.0</initial_velocity>
+        </plugin>
+        <plugin filename="gz-sim-joint-controller-system" name="gz::sim::systems::JointController">
+            <joint_name>joint5</joint_name>
+            <initial_velocity>5.0</initial_velocity>
+        </plugin>
+        <plugin filename="gz-sim-joint-controller-system" name="gz::sim::systems::JointController">
+            <joint_name>joint6</joint_name>
+            <initial_velocity>5.0</initial_velocity>
+        </plugin> -->
+        <!-- <plugin filename="ignition-gazebo-joint-position-controller-system" name="ignition::gazebo::systems::JointPositionController">
                 <joint_name>joint1</joint_name>
                 <p_gain>100.0</p_gain>
@@ -58,5 +177,5 @@
                 <i_max>-1.0</i_max>
                 <i_min>1.0</i_min>
-        </plugin>
+        </plugin> -->
         <plugin filename="ignition-gazebo-sensors-system" name="ignition::gazebo::systems::Sensors">
             <render_engine>ogre2</render_engine>

File: igus_rebel_description_ros2/urdf/igus_rebel/igus_rebel.urdf.xacro (robot description, xacro)
@@ -15,5 +15,6 @@
         </xacro:if>
         <!-- Gazebo macro -->
-        <xacro:include filename="$(find igus_rebel_description_ros2)/urdf/igus_rebel.gazebo.xacro" />
+        <xacro:include filename="$(find igus_rebel_description_ros2)/urdf/igus_rebel/igus_rebel.gazebo.xacro" />
+        <xacro:ign_ros2_control controller_parameters="$(find igus_rebel_moveit_config)/config/ros2_controllers.yaml"/>
     </xacro:macro>
 </robot>
