Commit message: gripper replaced with mount (camera in mount_v1), no tf for ignition bug but direclty link and joint, check if load base the ingition sensor plugin is not loaded (because in scout there is one already)

File: igus_rebel_description_ros2/urdf/igus_rebel/igus_rebel.gazebo.xacro (robot description, xacro)
@@ -23,5 +23,5 @@
     </xacro:macro>
     <!-- Sensor plugin -->
-    <xacro:macro name="virtual_sensors">
+     <xacro:macro name="ign_sensor_plugin">
         <gazebo>
             <plugin filename="ignition-gazebo-sensors-system" name="ignition::gazebo::systems::Sensors">
@@ -29,4 +29,23 @@
             </plugin>
         </gazebo>
+    </xacro:macro>
+    <!-- Ignition sensors -->
+    <xacro:macro name="virtual_sensors">
+        <!-- Optical frame id for depth image sensor -->
+        <joint name="camera_link_to_depth_image" type="fixed">
+            <parent link="camera_link" />
+            <child link="igus_rebel/link_8/depth_camera" />
+            <origin rpy="${-pi/2} 0.0 ${-pi/2}" xyz="0.0 0.0 0.0" />
+            <axis xyz="0 0 0" />
+        </joint>
+        <link name="igus_rebel/link_8/depth_camera" />
+        <!-- Optical frame id for pointcloud sensor -->
+        <joint name="camera_link_to_pointcloud" type="fixed">
+            <parent link="camera_link" />
+            <child link="igus_rebel/link_8/pointcloud" />
+            <origin rpy="0.0 0.0 0.0" xyz="0.0 0.0 0.0" />
+            <axis xyz="0 0 0" />
+        </joint>
+        <link name="igus_rebel/link_8/pointcloud" />
         <!-- Sensor for RGB, depth and pointcloud data -->
         <gazebo reference="virtual_rgb_camera_frame">

File: igus_rebel_description_ros2/urdf/igus_rebel/igus_rebel.urdf.xacro (robot description, xacro)
@@ -2,5 +2,5 @@
 <robot xmlns:xacro="http://www.ros.org/wiki/xacro" name="igus_rebel">
     <!-- macro definition for the robot -->
-    <xacro:macro name="igus_rebel" params="gripper camera end_effector hardware_protocol load_gazebo moveit">
+    <xacro:macro name="igus_rebel" params="load_base mount camera end_effector hardware_protocol load_gazebo moveit">
         <!-- Include and call rebel macro -->
         <xacro:include filename="$(find igus_rebel_description_ros2)/urdf/igus_rebel/igus_rebel.description.xacro" />
@@ -9,8 +9,8 @@
         <xacro:include filename="$(find igus_rebel_description_ros2)/urdf/igus_rebel/igus_rebel.control.xacro" />
         <xacro:igus_rebel_control hardware_protocol="${hardware_protocol}" />
-        <!-- Gripper macro -->
-        <xacro:if value="${gripper == 'camera'}">
-            <xacro:include filename="$(find igus_rebel_description_ros2)/urdf/grippers/grippers.xacro"/>
-            <xacro:gripper camera="$(arg camera)" end_effector="$(arg end_effector)" load_gazebo="$(arg load_gazebo)"/>
+        <!-- Mount macro -->
+        <xacro:if value="${mount == 'mount_v1'}">
+            <xacro:include filename="$(find igus_rebel_description_ros2)/urdf/mounts/mount_v1.xacro"/>
+            <xacro:mount_v1 camera="$(arg camera)" end_effector="$(arg end_effector)" load_gazebo="$(arg load_gazebo)"/>
         </xacro:if>
         <!-- Gazebo macro -->
@@ -23,6 +23,9 @@
                 <xacro:ign_joint_state_publisher/>
             </xacro:unless>
-            <xacro:unless value="${camera == 'none' or gripper == 'none'}">
+            <xacro:unless value="${camera == 'none' or mount == 'none'}">
                 <xacro:virtual_sensors/>
+                <xacro:unless value="${load_base}">
+                    <xacro:ign_sensor_plugin/>
+                </xacro:unless>
             </xacro:unless>
         </xacro:if>

File: igus_rebel_description_ros2/urdf/robot.urdf.xacro (robot description, xacro)
@@ -3,7 +3,6 @@
     <!-- Scout base selection -->
     <xacro:arg name="load_base" default="true" />
-    <!-- Gripper selection -->
-    <!-- CHANGE IN MOUNT and the options are V1, V2, .. -->
-    <xacro:arg name="gripper" default="none" />
+    <!-- Mount selection -->
+    <xacro:arg name="mount" default="none" />
     <!-- Camera type selection -->
     <xacro:arg name="camera" default="none" />
@@ -69,9 +68,9 @@
         </joint>
     </xacro:unless>
-    <!-- load igus rebel with camera gripper and castle -->
+    <!-- load igus rebel -->
     <xacro:include
         filename="$(find igus_rebel_description_ros2)/urdf/igus_rebel/igus_rebel.urdf.xacro" />
     <xacro:igus_rebel
-            gripper="$(arg gripper)" camera="$(arg camera)" end_effector="$(arg end_effector)"
+            load_base="$(arg load_base)" mount="$(arg mount)" camera="$(arg camera)" end_effector="$(arg end_effector)"
         hardware_protocol="$(arg hardware_protocol)" load_gazebo="$(arg load_gazebo)" moveit="$(arg moveit)" />
 </robot>

File: igus_rebel_moveit_config/config/igus_rebel.srdf.xacro (robot description, xacro)
@@ -3,12 +3,12 @@
 	<!-- Arguments -->
 	<xacro:arg name="load_base" default="false" />
-	<xacro:arg name="gripper" default="none" />
+	<xacro:arg name="mount" default="none" />
 	<xacro:arg name="camera" default="none" />
 	<xacro:arg name="end_effector" default="none" />
-	<!-- macro xacro definition to load gripper and mobile robot base -->
-	<xacro:macro name="srdf" params="gripper camera end_effector load_base">
+	<!-- macro xacro definition to load mount and mobile robot base -->
+	<xacro:macro name="srdf" params="mount camera end_effector load_base">
 		<!-- Groups -->
-		<!-- If gripper is not placed -->
-		<xacro:if value="${gripper == 'none'}">
+		<!-- If mount is not placed -->
+		<xacro:if value="${mount == 'none'}">
 			<group name="rebel_arm">
 				<chain base_link="igus_rebel_base_link" tip_link="link_8" />
@@ -19,6 +19,6 @@
 			<end_effector name="flange_EEF" parent_link="link_8" group="flange_group" parent_group="rebel_arm"/>
 		</xacro:if>
-		<!-- If gripper is placed -->
-		<xacro:if value="${gripper == 'camera'}">
+		<!-- If mount is placed -->
+		<xacro:if value="${mount == 'mount_v1'}">
 			<!-- If camera is none and no end effector -->
 			<xacro:if value="${camera == 'none' and end_effector == 'none'}">
@@ -180,6 +180,6 @@
 			<disable_collisions link1="rear_right_wheel_link" link2="tower_link" reason="Never"/>
 		</xacro:if>
-		<!-- Collision checks due to the presence of the gripper -->
-		<xacro:if value="${gripper == 'camera'}">
+		<!-- Collision checks due to the presence of the mount -->
+		<xacro:if value="${mount == 'mount_v1'}">
 			<disable_collisions link1="link_5" link2="camera_mount" reason="Never" />
 			<disable_collisions link1="link_6" link2="camera_mount" reason="Never" />
@@ -255,4 +255,4 @@
 	</xacro:macro>
 	<!-- Call the macro and define the arguments -->
-	<xacro:srdf gripper="$(arg gripper)" camera="$(arg camera)" end_effector="$(arg end_effector)" load_base="$(arg load_base)" />
+	<xacro:srdf mount="$(arg mount)" camera="$(arg camera)" end_effector="$(arg end_effector)" load_base="$(arg load_base)" />
 </robot>
