Commit message: added robot.urdf and scout from agilex pack, work on descr and moveit, bug wheels

File: igus_rebel_description_ros2/urdf/grippers/grippers.xacro (robot description, xacro)
@@ -5,5 +5,5 @@
         <color rgba="${5/255.0} ${15/255.0} ${5/255.0} 1.000" />
     </material>
-    <xacro:macro name="gripper" params="camera_type">
+    <xacro:macro name="gripper" params="camera">
         <!-- links the flange on the last joint to the gripper mount -->
         <joint name="flange_to_mount" type="fixed">
@@ -51,5 +51,5 @@
         </joint>
         <link name="camera_insert" />
-        <xacro:if value="${camera_type == 'realsense'}">
+        <xacro:if value="${camera == 'realsense'}">
             <!-- includes the realsense D435 ros2 description file and its collision box-->
             <xacro:arg name="use_nominal_extrinsics" default="false" />
@@ -62,4 +62,8 @@
             </xacro:sensor_d435>
         </xacro:if>
+        <xacro:if value="${camera == 'oakd'}">
+                <xacro:include filename="$(find igus_rebel_description_ros2)/urdf/camera/oak_d_pro.xacro"/>
+                <xacro:oakd_link/>
+        </xacro:if>
     </xacro:macro>
 </robot>

File: igus_rebel_description_ros2/urdf/igus_rebel/igus_rebel.description.xacro (robot description, xacro)
@@ -8,10 +8,10 @@
         <xacro:property name="damping" value="0.1"/>
         <xacro:property name="friction" value="10.0"/>
-        <link name="base_link">
+        <link name="igus_rebel_base_link">
             <visual>
                 <geometry>
                     <mesh filename="file://$(find igus_rebel_description_ros2)/meshes/new/Joint0.dae" />
                 </geometry>
-				<material name="dark_grey"/>
+                <material name="dark_grey"/>
             </visual>
             <collision>
@@ -26,5 +26,5 @@
         </link>
         <joint name="joint1" type="revolute">
-            <parent link="base_link" />
+            <parent link="igus_rebel_base_link" />
             <child link="link_1" />
             <origin rpy="0.0 0.0 0.0" xyz="0.0 0 0.100" />
@@ -39,5 +39,5 @@
                 </geometry>
                 <origin rpy="0 0 0" xyz="0 0 0" />
-				<material name="dark_grey"/>
+                <material name="dark_grey"/>
             </visual>
             <collision>
@@ -67,5 +67,5 @@
                 </geometry>
                 <origin rpy="0 0 0" xyz="0 0 0" />
-				<material name="dark_grey"/>
+                <material name="dark_grey"/>
             </visual>
             <collision>
@@ -95,5 +95,5 @@
                 </geometry>
                 <origin rpy="0 0 0" xyz="0 0 0" />
-				<material name="dark_grey"/>
+                <material name="dark_grey"/>
             </visual>
             <collision>
@@ -123,5 +123,5 @@
                 </geometry>
                 <origin rpy="0 0 0" xyz="0 0 0" />
-				<material name="dark_grey"/>
+                <material name="dark_grey"/>
             </visual>
             <collision>
@@ -151,5 +151,5 @@
                 </geometry>
                 <origin rpy="0 0 0" xyz="0 0 0" />
-				<material name="dark_grey"/>
+                <material name="dark_grey"/>
             </visual>
             <collision>
@@ -178,5 +178,5 @@
                 </geometry>
                 <origin rpy="0 0 0" xyz="0.0 0 0" />
-				<material name="dark_grey"/>
+                <material name="dark_grey"/>
             </visual>
             <collision>

File: igus_rebel_moveit_config/config/igus_rebel.srdf.xacro (robot description, xacro)
@@ -23,5 +23,5 @@
 		<!-- common definitions -->
 		<group name="rebel_arm">
-			<link name="base_link" />
+			<link name="igus_rebel_base_link" />
 			<link name="link_1" />
 			<link name="link_2" />
@@ -34,5 +34,5 @@
 		<xacro:if value="${gripper == 'none'}">
 			<group name="chain_arm">
-				<chain base_link="base_link" tip_link="link_8" />
+				<chain base_link="igus_rebel_base_link" tip_link="link_8" />
 			</group>
 			<end_effector name="manipulator" parent_link="link_8" group="rebel_arm" parent_group="chain_arm" />
@@ -50,5 +50,5 @@
 			</group>
 			<group name="chain_arm_manipulator">
-				<chain base_link="base_link" tip_link="toucher" />
+				<chain base_link="igus_rebel_base_link" tip_link="toucher" />
 			</group>
 			<end_effector name="manipulator" parent_link="toucher" group="chain_arm_manipulator"
@@ -92,6 +92,7 @@
 		<virtual_joint name="world_to_base" type="fixed" parent_frame="world" child_link="base_link" />
 		<!-- default collision checks for base robot -->
-		<disable_collisions link1="base_link" link2="link_1" reason="Adjacent" />
-		<disable_collisions link1="base_link" link2="link_2" reason="Never" />
+		<disable_collisions link1="base_link" link2="igus_rebel_base_link" reason="Adjacent" />
+		<disable_collisions link1="igus_rebel_base_link" link2="link_1" reason="Adjacent" />
+		<disable_collisions link1="igus_rebel_base_link" link2="link_2" reason="Never" />
 		<disable_collisions link1="link_1" link2="link_2" reason="Adjacent" />
 		<disable_collisions link1="link_2" link2="link_5" reason="Adjacent" />
@@ -112,5 +113,5 @@
 			<disable_collisions link1="camera_link" link2="toucher" reason="Never" />
 			<disable_collisions link1="camera_mount" link2="toucher" reason="Never" />
-			<xacro:no_collision_camera link="base_link" />
+			<xacro:no_collision_camera link="igus_rebel_base_link" />
 			<xacro:no_collision_camera link="link_1" />
 			<xacro:no_collision_camera link="link_2" />
@@ -134,10 +135,10 @@
 				<link name="tower_link" />
 			</group>
-			<disable_collisions link1="base_link" link2="front_left_wheel_link" reason="Never" />
-			<disable_collisions link1="base_link" link2="front_right_wheel_link" reason="Never" />
-			<disable_collisions link1="base_link" link2="mobile_robot_base_link" reason="Adjacent" />
-			<disable_collisions link1="base_link" link2="rear_left_wheel_link" reason="Never" />
-			<disable_collisions link1="base_link" link2="rear_right_wheel_link" reason="Never" />
-			<disable_collisions link1="base_link" link2="tower_link" reason="Never" />
+			<disable_collisions link1="igus_rebel_base_link" link2="front_left_wheel_link" reason="Never" />
+			<disable_collisions link1="igus_rebel_base_link" link2="front_right_wheel_link" reason="Never" />
+			<disable_collisions link1="igus_rebel_base_link" link2="mobile_robot_base_link" reason="Adjacent" />
+			<disable_collisions link1="igus_rebel_base_link" link2="rear_left_wheel_link" reason="Never" />
+			<disable_collisions link1="igus_rebel_base_link" link2="rear_right_wheel_link" reason="Never" />
+			<disable_collisions link1="igus_rebel_base_link" link2="tower_link" reason="Never" />
 			<disable_collisions link1="front_left_wheel_link" link2="front_right_wheel_link" reason="Never" />
 			<disable_collisions link1="front_left_wheel_link" link2="link_1" reason="Never" />

Commit message: virtual camera frames, ign_control and jsp based on visualzie and moveit launch,

File: igus_rebel_description_ros2/urdf/grippers/grippers.xacro (robot description, xacro)
@@ -5,5 +5,5 @@
         <color rgba="${5/255.0} ${15/255.0} ${5/255.0} 1.000" />
     </material>
-    <xacro:macro name="gripper" params="camera">
+    <xacro:macro name="gripper" params="camera load_gazebo">
         <!-- links the flange on the last joint to the gripper mount -->
         <joint name="flange_to_mount" type="fixed">
@@ -51,5 +51,10 @@
         </joint>
         <link name="camera_insert" />
+        <!-- Cameras -->
         <xacro:if value="${camera == 'realsense'}">
+            <xacro:if value="${load_gazebo}">
+                <xacro:include filename="$(find igus_rebel_description_ros2)/urdf/camera/virtual_camera_frames.xacro"/>
+                <xacro:virtual_camera_frames/>
+            </xacro:if>
             <!-- includes the realsense D435 ros2 description file and its collision box-->
             <xacro:arg name="use_nominal_extrinsics" default="false" />
@@ -63,6 +68,10 @@
         </xacro:if>
         <xacro:if value="${camera == 'oakd'}">
-                <xacro:include filename="$(find igus_rebel_description_ros2)/urdf/camera/oak_d_pro.xacro"/>
-                <xacro:oakd_link/>
+                <xacro:if value="${load_gazebo}">
+                    <xacro:include filename="$(find igus_rebel_description_ros2)/urdf/camera/virtual_camera_frames.xacro"/>
+                    <xacro:virtual_camera_frames/>
+                </xacro:if>
+                <xacro:include filename="$(find igus_rebel_description_ros2)/urdf/camera/oak_d_pro_camera.xacro"/>
+                <xacro:oak_d_pro_camera/>
         </xacro:if>
     </xacro:macro>

File: igus_rebel_description_ros2/urdf/igus_rebel/igus_rebel.gazebo.xacro (robot description, xacro)
@@ -1,4 +1,5 @@
 <?xml version="1.0"?>
 <robot xmlns:xacro="http://www.ros.org/wiki/xacro" name="igus_rebel_gazebo">
+    <!-- Ignition control plugin -->
     <xacro:macro name="ign_ros2_control" params="controller_parameters">
         <gazebo>
@@ -8,4 +9,18 @@
         </gazebo>
     </xacro:macro>
+    <!-- Joint state publisher plugin -->
+    <xacro:macro name="ign_joint_state_publisher">
+        <gazebo>
+            <plugin filename="ignition-gazebo-joint-state-publisher-system" name="ignition::gazebo::systems::JointStatePublisher">
+                <joint_name>joint1</joint_name>
+                <joint_name>joint2</joint_name>
+                <joint_name>joint3</joint_name>
+                <joint_name>joint4</joint_name>
+                <joint_name>joint5</joint_name>
+                <joint_name>joint6</joint_name>
+            </plugin>
+        </gazebo>
+    </xacro:macro>
+    <!-- Sensor plugin -->
     <gazebo>
         <plugin filename="ignition-gazebo-sensors-system" name="ignition::gazebo::systems::Sensors">
@@ -13,3 +28,82 @@
         </plugin>
     </gazebo>
+    <gazebo reference="virtual_rgb_camera_frame">
+        <sensor type="camera" name="rgb_camera">
+            <camera>
+                <horizontal_fov>1.05</horizontal_fov>
+                <image>
+                    <width>1280</width>
+                    <height>720</height>
+                </image>
+                <clip>
+                    <near>0.3</near>
+                    <far>100</far>
+                </clip>
+                <optical_frame_id>virtual_rgb_camera_frame</optical_frame_id>
+            </camera>
+            <always_on>1</always_on>
+            <update_rate>30</update_rate>
+            <visualize>true</visualize>
+        </sensor>
+    </gazebo>
+    <gazebo reference="virtual_depth_camera_frame">
+        <sensor type="rgbd_camera" name="depth_camera">
+            <update_rate>10</update_rate>
+            <depth_camera>
+                <horizontal_fov>1.05</horizontal_fov>
+                <image>
+                    <width>320</width>
+                    <height>240</height>
+                    <!-- <width>1280</width>
+                    <height>720</height> -->
+                    <format>R8G8B8</format>
+                </image>
+                <clip>
+                    <near>0.1</near>
+                    <far>10.0</far>
+                </clip>
+            </depth_camera>
+        </sensor>
+    </gazebo>
+    <gazebo reference="virtual_depth_camera_frame">
+        <sensor type="rgbd_camera" name="pointcloud">
+            <update_rate>10</update_rate>
+            <camera>
+                <horizontal_fov>1.05</horizontal_fov>
+                <image>
+                    <width>320</width>
+                    <height>240</height>
+                    <format>R8G8B8</format>
+                </image>
+                <clip>
+                    <near>0.1</near>
+                    <far>10.0</far>
+                </clip>
+            </camera>
+        </sensor>
+    </gazebo>
+    <!-- <gazebo reference="oakd_joint">
+        <preserveFixedJoint>true</preserveFixedJoint>
+    </gazebo>
+    <gazebo reference="oakd_rgb_camera_joint">
+        <preserveFixedJoint>true</preserveFixedJoint>
+    </gazebo>
+    <gazebo reference="oakd_rgb_camera_optical_joint">
+        <preserveFixedJoint>true</preserveFixedJoint>
+    </gazebo>
+    <gazebo reference="oakd_left_camera_joint">
+        <preserveFixedJoint>true</preserveFixedJoint>
+    </gazebo>
+    <gazebo reference="oakd_left_camera_optical_joint">
+        <preserveFixedJoint>true</preserveFixedJoint>
+    </gazebo>
+    <gazebo reference="oakd_right_camera_joint">
+        <preserveFixedJoint>true</preserveFixedJoint>
+    </gazebo>
+    <gazebo reference="oakd_right_camera_optical_joint">
+        <preserveFixedJoint>true</preserveFixedJoint>
+    </gazebo>
+    <gazebo reference="oakd_imu_joint">
+        <preserveFixedJoint>true</preserveFixedJoint>
+    </gazebo> -->
 </robot>

File: igus_rebel_description_ros2/urdf/igus_rebel/igus_rebel.urdf.xacro (robot description, xacro)
@@ -2,5 +2,5 @@
 <robot xmlns:xacro="http://www.ros.org/wiki/xacro" name="igus_rebel">
     <!-- macro definition for the robot -->
-    <xacro:macro name="igus_rebel" params="gripper camera end_effector hardware_protocol load_gazebo">
+    <xacro:macro name="igus_rebel" params="gripper camera end_effector hardware_protocol load_gazebo moveit">
         <!-- Include and call rebel macro -->
         <xacro:include filename="$(find igus_rebel_description_ros2)/urdf/igus_rebel/igus_rebel.description.xacro" />
@@ -12,9 +12,16 @@
         <xacro:if value="${gripper == 'camera'}">
             <xacro:include filename="$(find igus_rebel_description_ros2)/urdf/grippers/grippers.xacro"/>
-            <xacro:gripper camera="$(arg camera)"/>
+            <xacro:gripper camera="$(arg camera)" load_gazebo="$(arg load_gazebo)"/>
         </xacro:if>
         <!-- Gazebo macro -->
-        <xacro:include filename="$(find igus_rebel_description_ros2)/urdf/igus_rebel/igus_rebel.gazebo.xacro" />
-        <xacro:ign_ros2_control controller_parameters="$(find igus_rebel_moveit_config)/config/ros2_controllers.yaml"/>
+        <xacro:if value="${load_gazebo}">
+            <xacro:include filename="$(find igus_rebel_description_ros2)/urdf/igus_rebel/igus_rebel.gazebo.xacro" />
+            <xacro:if value="${moveit}">
+                <xacro:ign_ros2_control controller_parameters="$(find igus_rebel_moveit_config)/config/ros2_controllers.yaml"/>
+            </xacro:if>
+            <xacro:unless value="${moveit}">
+                <xacro:ign_joint_state_publisher/>
+            </xacro:unless>
+        </xacro:if>
     </xacro:macro>
 </robot>

File: igus_rebel_description_ros2/urdf/robot.urdf.xacro (robot description, xacro)
@@ -14,4 +14,6 @@
     <!-- Controller settings, only enable a single one in the launch file -->
     <xacro:arg name="hardware_protocol" default="simulation" />
+    <!-- Argument that tells if Moveit2 is used or not -->
+    <xacro:arg name="moveit" default="true" />
     <!-- odometry source: world ground truth or wheels encoders -->
     <xacro:arg name="odometry_source" default="ground_truth" />
@@ -72,4 +74,4 @@
     <xacro:igus_rebel
             gripper="$(arg gripper)" camera="$(arg camera)" end_effector="$(arg end_effector)"
-        hardware_protocol="$(arg hardware_protocol)" load_gazebo="$(arg load_gazebo)" />
+        hardware_protocol="$(arg hardware_protocol)" load_gazebo="$(arg load_gazebo)" moveit="$(arg moveit)" />
 </robot>

Commit message: added toucher cylinder end effector, changed camera in cameras folder, rewritten srdf file with good collisions and groups

File: igus_rebel_description_ros2/urdf/grippers/grippers.xacro (robot description, xacro)
@@ -5,5 +5,5 @@
         <color rgba="${5/255.0} ${15/255.0} ${5/255.0} 1.000" />
     </material>
-    <xacro:macro name="gripper" params="camera load_gazebo">
+    <xacro:macro name="gripper" params="camera end_effector load_gazebo">
         <!-- links the flange on the last joint to the gripper mount -->
         <joint name="flange_to_mount" type="fixed">
@@ -36,11 +36,4 @@
             </collision>
         </link>
-        <joint name="flange_to_toucher" type="fixed">
-            <parent link="flange" />
-            <child link="toucher" />
-            <origin rpy="0.0 0.0 0.0" xyz="0.1 0.0 0.0" /> <!-- 10 cm in front of the flange origin -->
-            <axis xyz="0 0 0" />
-        </joint>
-        <link name="toucher" />
         <!-- positions the camera inside the structure -->
         <joint name="mount_to_cam" type="fixed">
@@ -51,8 +44,13 @@
         </joint>
         <link name="camera_insert" />
+        <!-- End effectors -->
+        <xacro:if value="${end_effector == 'toucher_cylinder'}">
+            <xacro:include filename="$(find igus_rebel_description_ros2)/urdf/end_effectors/toucher_cylinder.xacro"/>
+            <xacro:toucher_cylinder parent="camera_mount"/>
+        </xacro:if>
         <!-- Cameras -->
         <xacro:if value="${camera == 'realsense'}">
             <xacro:if value="${load_gazebo}">
-                <xacro:include filename="$(find igus_rebel_description_ros2)/urdf/camera/virtual_camera_frames.xacro"/>
+                <xacro:include filename="$(find igus_rebel_description_ros2)/urdf/cameras/virtual_camera_frames.xacro"/>
                 <xacro:virtual_camera_frames/>
             </xacro:if>
@@ -68,10 +66,10 @@
         </xacro:if>
         <xacro:if value="${camera == 'oakd'}">
-                <xacro:if value="${load_gazebo}">
-                    <xacro:include filename="$(find igus_rebel_description_ros2)/urdf/camera/virtual_camera_frames.xacro"/>
-                    <xacro:virtual_camera_frames/>
-                </xacro:if>
-                <xacro:include filename="$(find igus_rebel_description_ros2)/urdf/camera/oak_d_pro_camera.xacro"/>
-                <xacro:oak_d_pro_camera/>
+            <xacro:if value="${load_gazebo}">
+                <xacro:include filename="$(find igus_rebel_description_ros2)/urdf/cameras/virtual_camera_frames.xacro"/>
+                <xacro:virtual_camera_frames/>
+            </xacro:if>
+            <xacro:include filename="$(find igus_rebel_description_ros2)/urdf/cameras/oak_d_pro_camera.xacro"/>
+            <xacro:oak_d_pro_camera/>
         </xacro:if>
     </xacro:macro>

File: igus_rebel_description_ros2/urdf/igus_rebel/igus_rebel.urdf.xacro (robot description, xacro)
@@ -12,5 +12,5 @@
         <xacro:if value="${gripper == 'camera'}">
             <xacro:include filename="$(find igus_rebel_description_ros2)/urdf/grippers/grippers.xacro"/>
-            <xacro:gripper camera="$(arg camera)" load_gazebo="$(arg load_gazebo)"/>
+            <xacro:gripper camera="$(arg camera)" end_effector="$(arg end_effector)" load_gazebo="$(arg load_gazebo)"/>
         </xacro:if>
         <!-- Gazebo macro -->
