Commit message: new mash color, damping zero, jpc for description, zero gravity, spawn args

File: igus_rebel_description_ros2/urdf/end_effectors/toucher_cylinder.xacro (robot description, xacro)
@@ -21,5 +21,7 @@
                     <cylinder length="0.225" radius="0.015" />
                 </geometry>
-                <material name="dark_green" />
+                <material name="toucher_cylinder_color">
+                    <color rgba="${5/255.0} ${5/255.0} ${5/255.0} 1.000" />
+                </material>
             </visual>
             <collision>

File: igus_rebel_description_ros2/urdf/igus_rebel/igus_rebel.description.xacro (robot description, xacro)
@@ -2,10 +2,10 @@
 <robot xmlns:xacro="http://www.ros.org/wiki/xacro" name="igus_rebel">
     <material name="dark_grey">
-        <color rgba="${5/255} ${5/255} ${5/255} 1.0" />
+        <color rgba="${5/255.0} ${5/255.0} ${5/255.0} 1.000" />
     </material>
     <xacro:macro name="igus_rebel_description">
         <!-- Set both at 0.0 if collapsing is not interesting in gazebo -->
-        <xacro:property name="damping" value="0.1"/>
-        <xacro:property name="friction" value="10.0"/>
+        <xacro:property name="damping" value="0.0"/>
+        <xacro:property name="friction" value="0.0"/>
         <link name="igus_rebel_base_link">
             <visual>

File: igus_rebel_description_ros2/urdf/igus_rebel/igus_rebel.gazebo.xacro (robot description, xacro)
@@ -1,4 +1,23 @@
 <?xml version="1.0"?>
 <robot xmlns:xacro="http://www.ros.org/wiki/xacro" name="igus_rebel_gazebo">
+    <!-- Colors -->
+    <gazebo reference="camera_mount">
+        <visual>
+            <material>
+                <ambient>0.03 0.03 0.03 1</ambient>
+                <diffuse>0.03 0.03 0.03 1</diffuse>
+                <specular>0.03 0.03 0.03 1</specular>
+            </material>
+        </visual>
+    </gazebo>
+    <gazebo reference="toucher_cylinder">
+        <visual>
+            <material>
+                <ambient>0.03 0.03 0.03 1</ambient>
+                <diffuse>0.03 0.03 0.03 1</diffuse>
+                <specular>0.03 0.03 0.03 1</specular>
+            </material>
+        </visual>
+    </gazebo>
     <!-- Ignition control plugin -->
     <xacro:macro name="ign_ros2_control" params="controller_parameters">
@@ -19,4 +38,57 @@
                 <joint_name>joint5</joint_name>
                 <joint_name>joint6</joint_name>
+            </plugin>
+        </gazebo>
+    </xacro:macro>
+    <!-- Joint position controller plugin -->
+    <xacro:macro name="ign_joint_position_controller">
+        <gazebo>
+            <plugin filename="ignition-gazebo-joint-position-controller-system" name="ignition::gazebo::systems::JointPositionController">
+                    <joint_name>joint1</joint_name>
+                    <p_gain>1000.0</p_gain>
+                    <i_gain>0.0</i_gain>
+                    <d_gain>50.0</d_gain>
+                    <i_max>-1.0</i_max>
+                    <i_min>1.0</i_min>
+            </plugin>
+            <plugin filename="ignition-gazebo-joint-position-controller-system" name="ignition::gazebo::systems::JointPositionController">
+                    <joint_name>joint2</joint_name>
+                    <p_gain>1000.0</p_gain>
+                    <i_gain>0.0</i_gain>
+                    <d_gain>50.0</d_gain>
+                    <i_max>-1.0</i_max>
+                    <i_min>1.0</i_min>
+            </plugin>
+            <plugin filename="ignition-gazebo-joint-position-controller-system" name="ignition::gazebo::systems::JointPositionController">
+                    <joint_name>joint3</joint_name>
+                    <p_gain>1000.0</p_gain>
+                    <i_gain>0.0</i_gain>
+                    <d_gain>50.0</d_gain>
+                    <i_max>-1.0</i_max>
+                    <i_min>1.0</i_min>
+            </plugin>
+            <plugin filename="ignition-gazebo-joint-position-controller-system" name="ignition::gazebo::systems::JointPositionController">
+                    <joint_name>joint4</joint_name>
+                    <p_gain>1000.0</p_gain>
+                    <i_gain>0.0</i_gain>
+                    <d_gain>50.0</d_gain>
+                    <i_max>-1.0</i_max>
+                    <i_min>1.0</i_min>
+            </plugin>
+            <plugin filename="ignition-gazebo-joint-position-controller-system" name="ignition::gazebo::systems::JointPositionController">
+                    <joint_name>joint5</joint_name>
+                    <p_gain>1000.0</p_gain>
+                    <i_gain>0.0</i_gain>
+                    <d_gain>50.0</d_gain>
+                    <i_max>-1.0</i_max>
+                    <i_min>1.0</i_min>
+            </plugin>
+            <plugin filename="ignition-gazebo-joint-position-controller-system" name="ignition::gazebo::systems::JointPositionController">
+                    <joint_name>joint6</joint_name>
+                    <p_gain>1000.0</p_gain>
+                    <i_gain>0.0</i_gain>
+                    <d_gain>50.0</d_gain>
+                    <i_max>-1.0</i_max>
+                    <i_min>1.0</i_min>
             </plugin>
         </gazebo>

File: igus_rebel_description_ros2/urdf/igus_rebel/igus_rebel.urdf.xacro (robot description, xacro)
@@ -22,4 +22,5 @@
             <xacro:unless value="${moveit}">
                 <xacro:ign_joint_state_publisher/>
+                <xacro:ign_joint_position_controller/>
             </xacro:unless>
             <xacro:unless value="${camera == 'none' or mount == 'none'}">

File: igus_rebel_description_ros2/urdf/mounts/mount_v1.xacro (robot description, xacro)
@@ -1,6 +1,6 @@
 <?xml version="1.0"?>
 <robot xmlns:xacro="http://www.ros.org/wiki/xacro" name="mount_v1">
-    <material name="dark_green">
-        <color rgba="${5/255.0} ${15/255.0} ${5/255.0} 1.000" />
+    <material name="mount_dark_grey">
+        <color rgba="${5/255.0} ${5/255.0} ${5/255.0} 1.000" />
     </material>
     <xacro:macro name="mount_v1" params="camera end_effector load_gazebo">
@@ -25,5 +25,7 @@
                         scale="0.001 0.001 0.001" />
                 </geometry>
-                <material name="dark_green" />
+                <material name="camera_mount_color">
+                    <color rgba="${5/255.0} ${5/255.0} ${5/255.0} 1.000" />
+                </material>
             </visual>
             <collision>

File: igus_rebel_description_ros2/urdf/robot.urdf.xacro (robot description, xacro)
@@ -18,6 +18,6 @@
     <xacro:arg name="odometry_source" default="ground_truth" />
     <!-- Set both at 0.0 if collapsing is not interesting in gazebo -->
-    <xacro:property name="damping" value="0.1"/>
-    <xacro:property name="friction" value="10.0"/>
+    <xacro:property name="damping" value="0.0"/>
+    <xacro:property name="friction" value="0.0"/>
     <!-- Load mobile robot base, load_base must be true -->
     <xacro:if value="$(arg load_base)">
